File: hw/Pulse_Fire.kicad_pcb (KiCad board)
At the start: 2 copper layers, 0 parts

Commit message: hw: Complete board design
Parts:
- added BT1: NiMH AAA, Battery:BatteryHolder_Keystone_2466_1xAAA, B.Cu at (172.3, 100.0)
- added C1: 100n, Capacitor_SMD:C_0402_1005Metric, F.Cu at (148.7, 102.6)
- added C10: 22u, Capacitor_SMD:C_0603_1608Metric, F.Cu at (162.3, 104.0)
- added C11: 220u, Capacitor_SMD:CP_Elec_6.3x5.4, F.Cu at (161.7, 83.3)
- added C12: 1u, Capacitor_SMD:C_0402_1005Metric, F.Cu at (157.8, 97.8)
- added C13: 1u, Capacitor_SMD:C_0402_1005Metric, F.Cu at (155.4, 100.0)
- added C2: 100n, Capacitor_SMD:C_0402_1005Metric, F.Cu at (153.2, 92.2)
- added C3: 100n, Capacitor_SMD:C_0402_1005Metric, F.Cu at (153.6, 95.8)
- added C4: 100n, Capacitor_SMD:C_0402_1005Metric, F.Cu at (144.0, 112.2)
- added C5: 1n, Capacitor_SMD:C_0402_1005Metric, F.Cu at (145.9, 113.2)
- added C6: 4.7u, Capacitor_SMD:C_0402_1005Metric, F.Cu at (150.2, 108.3)
- added C7: 4.7u, Capacitor_SMD:C_0402_1005Metric, F.Cu at (149.9, 116.7)
- added C8: 10u, Capacitor_SMD:C_0402_1005Metric, F.Cu at (170.2, 100.5)
- added C9: 22u, Capacitor_SMD:C_0603_1608Metric, F.Cu at (162.3, 102.5)
- added D2: LED_RGBA, Connector_JST:JST_PH_S4B-PH-SM4-TB_1x04-1MP_P2.00mm_Horizontal, F.Cu at (150.0, 75.5)
- added J2: Conn_01x04, TestPoints_P2.00:TestPoints_1x04_P2.00, F.Cu at (170.8, 112.0)
- added L1: 22uH, Inductor_SMD:L_Sunlord_SWPA4030S, F.Cu at (166.8, 100.0)
- added LS1: Speaker, Connector_JST:JST_PH_S2B-PH-SM4-TB_1x02-1MP_P2.00mm_Horizontal, F.Cu at (150.0, 124.5)
- added Q1: AO3400A, Package_TO_SOT_SMD:SOT-23, F.Cu at (154.0, 86.0)
- added Q2: AO3400A, Package_TO_SOT_SMD:SOT-23, F.Cu at (150.0, 86.0)
- added Q3: AO3400A, Package_TO_SOT_SMD:SOT-23, F.Cu at (146.0, 86.0)
- added R1: 68, Resistor_SMD:R_0603_1608Metric, F.Cu at (154.0, 82.6)
- added R2: 47, Resistor_SMD:R_0603_1608Metric, F.Cu at (150.0, 82.6)
- added R3: 47, Resistor_SMD:R_0603_1608Metric, F.Cu at (146.0, 82.6)
- added R4: 100k, Resistor_SMD:R_0402_1005Metric, F.Cu at (144.9, 111.3)
- added R5: 22k, Resistor_SMD:R_0402_1005Metric, F.Cu at (145.9, 112.2)
- added U1: PY32F003F18U6, Package_DFN_QFN:QFN-20-1EP_3x3mm_P0.4mm_EP1.65x1.65mm, F.Cu at (150.0, 100.0)
- added U2: SC7A20, Package_LGA:LGA-12_2x2mm_P0.5mm, F.Cu at (152.8, 94.0)
- added U3: FM8002A, Package_SO:SOP-8_3.9x4.9mm_P1.27mm, F.Cu at (150.0, 112.5)
- added U4: ME6206A33XG, Package_TO_SOT_SMD:SOT-23, F.Cu at (157.8, 100.0)
- added U6: ME2188A50, Package_TO_SOT_SMD:SOT-23, F.Cu at (162.4, 100.0)
Routing:
- net +5V: track 0.00 -> 55.9 mm
- net +3V3: track 0.00 -> 40.2 mm, vias 0 -> 4
- net /SWDIO: track 0.00 -> 25.4 mm
- net /SWCLK: track 0.00 -> 25.3 mm
- net /AUDIO_OUT: track 0.00 -> 15.2 mm
- net /LED_B: track 0.00 -> 14.3 mm
- net /LED_R: track 0.00 -> 13.2 mm
- net /LED_G: track 0.00 -> 13.1 mm
- net /AUDIO_SD: track 0.00 -> 11.4 mm
- net Net-(U3-VO1): track 0.00 -> 10.5 mm
- net /IMU_INT1: track 0.00 -> 7.36 mm
- net Net-(U3-VO2): track 0.00 -> 6.90 mm
- net /IMU_CS: track 0.00 -> 6.49 mm
- net Net-(U3--IN): track 0.00 -> 5.34 mm
- net /IMU_SCK: track 0.00 -> 5.23 mm
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- added copper zone on B.Cu, net GND
- added copper zone on F.Cu, net GND
Other:
- board outline added: 60 x 60 mm
- board text added: "Added MP"
